Commit message: add panda_arm_EE move_group that has correct end effector for moveit

File: franka_description/robots/panda_arm.xacro (robot description, xacro)
@@ -208,4 +208,11 @@
       <axis xyz="0 0 0"/>
     </joint>
+    <link name="${arm_id}_EE"/>
+    <joint name="${arm_id}_jointEE" type="fixed">
+      <origin rpy="0 0 0.78539816339" xyz="0 0 0.1034"/>
+      <parent link="${arm_id}_link8"/>
+      <child link="${arm_id}_EE"/>
+      <axis xyz="0 0 0"/>
+    </joint>
   </xacro:macro>
 </robot>
